File: Hardware/Cyclope.sch (KiCad schematic (older format))
At the start: 4 parts

Commit message: [Hardware] Indicated all mechanical parts that must not be populated.
Parts:
- H10, H7, H8, H9: Populate (none) -> DNP
Changed lines of the file:
@@
 F 2 "MountingHole:MountingHole_3.2mm_M3_Pad" H 2050 6800 50  0001 C CNN
 F 3 "~" H 2050 6800 50  0001 C CNN
+F 4 "DNP" H 2050 6800 50  0001 C CNN "Populate"
 	1    2050 6800
 	1    0    0    -1
@@
 F 2 "MountingHole:MountingHole_3.2mm_M3_Pad" H 2750 6800 50  0001 C CNN
 F 3 "~" H 2750 6800 50  0001 C CNN
+F 4 "DNP" H 2750 6800 50  0001 C CNN "Populate"
 	1    2750 6800
 	1    0    0    -1
@@
 F 2 "MountingHole:MountingHole_3.2mm_M3_Pad" H 3450 6800 50  0001 C CNN
 F 3 "~" H 3450 6800 50  0001 C CNN
+F 4 "DNP" H 3450 6800 50  0001 C CNN "Populate"
 	1    3450 6800
 	1    0    0    -1
@@
 F 2 "MountingHole:MountingHole_3.2mm_M3_Pad" H 4150 6800 50  0001 C CNN
 F 3 "~" H 4150 6800 50  0001 C CNN
+F 4 "DNP" H 4150 6800 50  0001 C CNN "Populate"
 	1    4150 6800
 	1    0    0    -1
