File: Hardware/Front_Board.sch (KiCad schematic (older format))
At the start: 27 parts, among them J4 Front, J5 Front, Q1 DMG3414U

Commit message: [Hardware] Indicated all mechanical parts that must not be populated.
Parts:
- BT1, BT2, BT3, BT4, BT5, BT6, H11, H12, H3, H4, H5, H6: Populate (none) -> DNP
Changed lines of the file:
@@
 F 2 "MountingHole:MountingHole_2.2mm_M2" H 4500 2350 50  0001 C CNN
 F 3 "~" H 4500 2350 50  0001 C CNN
+F 4 "DNP" H 4500 2350 50  0001 C CNN "Populate"
 	1    4500 2350
 	1    0    0    -1
@@
 F 2 "MountingHole:MountingHole_2.2mm_M2" H 5250 2350 50  0001 C CNN
 F 3 "~" H 5250 2350 50  0001 C CNN
+F 4 "DNP" H 5250 2350 50  0001 C CNN "Populate"
 	1    5250 2350
 	1    0    0    -1
@@
 F 2 "MountingHole:MountingHole_2.2mm_M2" H 4500 2650 50  0001 C CNN
 F 3 "~" H 4500 2650 50  0001 C CNN
+F 4 "DNP" H 4500 2650 50  0001 C CNN "Populate"
 	1    4500 2650
 	1    0    0    -1
@@
 F 2 "MountingHole:MountingHole_2.2mm_M2" H 5250 2650 50  0001 C CNN
 F 3 "~" H 5250 2650 50  0001 C CNN
+F 4 "DNP" H 5250 2650 50  0001 C CNN "Populate"
 	1    5250 2650
 	1    0    0    -1
@@
 F 2 "MountingHole:MountingHole_3.2mm_M3" H 4500 2950 50  0001 C CNN
 F 3 "~" H 4500 2950 50  0001 C CNN
+F 4 "DNP" H 4500 2950 50  0001 C CNN "Populate"
 	1    4500 2950
 	1    0    0    -1
@@
 F 2 "MountingHole:MountingHole_3.2mm_M3" H 5250 2950 50  0001 C CNN
 F 3 "~" H 5250 2950 50  0001 C CNN
+F 4 "DNP" H 5250 2950 50  0001 C CNN "Populate"
 	1    5250 2950
 	1    0    0    -1
@@
 F 2 "Break_Tab:Break_Tab" H 5550 4300 50  0001 C CNN
 F 3 "~" H 5550 4300 50  0001 C CNN
+F 4 "DNP" H 5550 4300 50  0001 C CNN "Populate"
 	1    5550 4300
 	1    0    0    -1
@@
 F 2 "Break_Tab:Break_Tab" H 5550 4550 50  0001 C CNN
 F 3 "~" H 5550 4550 50  0001 C CNN
+F 4 "DNP" H 5550 4550 50  0001 C CNN "Populate"
 	1    5550 4550
 	1    0    0    -1
@@
 F 2 "Break_Tab:Break_Tab" H 5550 4800 50  0001 C CNN
 F 3 "~" H 5550 4800 50  0001 C CNN
+F 4 "DNP" H 5550 4800 50  0001 C CNN "Populate"
 	1    5550 4800
 	1    0    0    -1
@@
 F 2 "Break_Tab:Break_Tab" H 6800 4300 50  0001 C CNN
 F 3 "~" H 6800 4300 50  0001 C CNN
+F 4 "DNP" H 6800 4300 50  0001 C CNN "Populate"
 	1    6800 4300
 	1    0    0    -1
@@
 F 2 "Break_Tab:Break_Tab" H 6800 4550 50  0001 C CNN
 F 3 "~" H 6800 4550 50  0001 C CNN
+F 4 "DNP" H 6800 4550 50  0001 C CNN "Populate"
 	1    6800 4550
 	1    0    0    -1
@@
 F 2 "Break_Tab:Break_Tab" H 6800 4800 50  0001 C CNN
 F 3 "~" H 6800 4800 50  0001 C CNN
+F 4 "DNP" H 6800 4800 50  0001 C CNN "Populate"
 	1    6800 4800
 	1    0    0    -1
