File: Hardware/Power_Supply.sch (KiCad schematic (older format))
At the start: 16 parts, among them SW1 1101M2S3AQE2, U1 TPS565208DDC

Commit message: [Hardware] Indicated all mechanical parts that must not be populated.
Parts:
- C1, C5, C6, C7: ManufacturerReference CC1206KRX7R9BB104 -> (none)
- H1, H2: Populate (none) -> DNP
Changed lines of the file:
@@
 F 4 "25V" H 8585 3795 50  0000 R CNN "Value2"
 F 5 "X7R" H 8585 3886 50  0000 R CNN "Value3"
-F 6 "CC1206KRX7R9BB104" V 8700 3750 50  0001 C CNN "ManufacturerReference"
 	1    8700 3750
 	-1   0    0    1
@@
 F 4 "25V" H 9035 3795 50  0000 R CNN "Value2"
 F 5 "X7R" H 9035 3886 50  0000 R CNN "Value3"
-F 6 "CC1206KRX7R9BB104" V 9150 3750 50  0001 C CNN "ManufacturerReference"
 	1    9150 3750
 	-1   0    0    1
@@
 F 4 "25V" H 9485 3795 50  0000 R CNN "Value2"
 F 5 "X7R" H 9485 3886 50  0000 R CNN "Value3"
-F 6 "CC1206KRX7R9BB104" V 9600 3750 50  0001 C CNN "ManufacturerReference"
 	1    9600 3750
 	-1   0    0    1
@@
 F 2 "MountingHole:MountingHole_2.2mm_M2_Pad" H 2250 4000 50  0001 C CNN
 F 3 "~" H 2250 4000 50  0001 C CNN
+F 4 "DNP" H 2250 4000 50  0001 C CNN "Populate"
 	1    2250 4000
 	0    -1   -1   0
@@
 F 2 "MountingHole:MountingHole_2.2mm_M2_Pad" H 2250 3400 50  0001 C CNN
 F 3 "~" H 2250 3400 50  0001 C CNN
+F 4 "DNP" H 2250 3400 50  0001 C CNN "Populate"
 	1    2250 3400
 	0    -1   -1   0
@@
 F 4 "25V" V 6550 3700 50  0000 C CNN "Value2"
 F 5 "X7R" V 6650 3700 50  0000 C CNN "Value3"
-F 6 "CC1206KRX7R9BB104" V 6900 3700 50  0001 C CNN "ManufacturerReference"
 	1    6900 3700
 	0    1    1    0
