File: Hardware/Lidar.sch (KiCad schematic (older format))
At the start: 9 parts, among them J6 22-03-5075, Q6 DMG2301L, Q7 DMG3414U

Commit message: [Hardware] Indicated all mechanical parts that must not be populated.
Parts:
- C22: ManufacturerReference CC1206KRX7R9BB104 -> (none)
Changed lines of the file:
@@
 F 4 "25V" H 4685 4295 50  0000 R CNN "Value2"
 F 5 "X7R" H 4685 4386 50  0000 R CNN "Value3"
-F 6 "CC1206KRX7R9BB104" V 4800 4250 50  0001 C CNN "ManufacturerReference"
 	1    4800 4250
 	-1   0    0    1

Commit message: [Hardware] Mirrored lidar connector as connector datasheet numbering does not match lidar datasheet numbering.
Connections:
- net GND: now also J6.1 (Pin_1), J6.5 (Pin_5); no longer J6.3 (Pin_3), J6.7 (Pin_7)
- net LIDAR_UART_RX: now also J6.2 (Pin_2); no longer J6.6 (Pin_6)
- net LIDAR_UART_TX: now also J6.3 (Pin_3); no longer J6.5 (Pin_5)
- net at C21.1, C22.2, Q6.3 (D)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: now also J6.6 (Pin_6), J6.7 (Pin_7); no longer J6.1 (Pin_1), J6.2 (Pin_2)
Changed lines of the file:
@@
 	1    0    0    -1
-$EndComp
-$Comp
-L Connector_Generic:Conn_01x07 J?
-U 1 1 60342521
-P 6100 2150
-AR Path="/5F22814A/60342521" Ref="J?"  Part="1"
-AR Path="/601E5913/60342521" Ref="J6"  Part="1"
-F 0 "J6" V 6064 1762 50  0000 R CNN
-F 1 "22-03-5075" V 5973 1762 50  0000 R CNN
-F 2 "Connector_Molex:Molex_SPOX_5267-07A_1x07_P2.50mm_Vertical" H 6100 2150 50  0001 C CNN
-F 3 "https://www.molex.com/webdocs/datasheets/pdf/en-us/0022035075_PCB_HEADERS.pdf" H 6100 2150 50  0001 C CNN
-F 4 "Molex" H 6100 2150 50  0001 C CNN "Manufacturer"
-	1    6100 2150
-	0    -1   -1   0
 $EndComp
 Text Notes 5800 1950 0    50   ~ 0
@@
 Text Notes 4850 5200 0    50   ~ 0
 Allow to create a pi\nfilter if needed to keep\nlidar core voltage below\n50mVpp ripple.
+$Comp
+L Connector_Generic:Conn_01x07 J?
+U 1 1 60342521
+P 6100 2150
+AR Path="/5F22814A/60342521" Ref="J?"  Part="1"
+AR Path="/601E5913/60342521" Ref="J6"  Part="1"
+F 0 "J6" V 6064 2530 50  0000 L CNN
+F 1 "22-03-5075" V 5973 2530 50  0000 L CNN
+F 2 "Connector_Molex:Molex_SPOX_5267-07A_1x07_P2.50mm_Vertical" H 6100 2150 50  0001 C CNN
+F 3 "https://www.molex.com/webdocs/datasheets/pdf/en-us/0022035075_PCB_HEADERS.pdf" H 6100 2150 50  0001 C CNN
+F 4 "Molex" H 6100 2150 50  0001 C CNN "Manufacturer"
+	1    6100 2150
+	0    1    -1   0
+$EndComp
 $EndSCHEMATC
